Commit message: Fix: remove nested git repo and vendor rf2o_laser_odometry

File: src/ika_description/urdf/ika.xacro (robot description, xacro)
@@ -27,8 +27,8 @@
 </link>
 <!-- Lidar (RPLidar S2) -->
-<xacro:rplidar_s2 parent="base_link" name="lidar" xyz="1.07 -0.015 0.63" rpy="0 0.035 0"/>
+<xacro:rplidar_s2 parent="base_link" name="lidar" xyz="0.2 0 0.36" rpy="0 0.035 0"/>
 <xacro:rplidar_s2_gazebo_plugin name="lidar"/>
 <!-- Kamera (D435) -->
-<xacro:realsense_d435 parent="base_link" name="camera" xyz="0.46 -0.10 0.985" rpy="0 0 0"/>
+<xacro:realsense_d435 parent="base_link" name="camera" xyz="0.2 -0.10 0.37" rpy="0 0 0"/>
 <xacro:d435_gazebo_plugins name="camera"/>
 <link name="lazer_alt_v1_1">
@@ -352,5 +352,5 @@
   </collision>
 </link>
-<joint name="laser_alt" type="continuous">
+<joint name="laser_alt" type="fixed">
   <origin xyz="0.000155 -0.001158 0.366945" rpy="0 0 0"/>
   <parent link="base_link"/>
@@ -358,5 +358,5 @@
   <axis xyz="0.0 0.0 1.0"/>
 </joint>
-<joint name="laser_ust" type="revolute">
+<joint name="laser_ust" type="fixed">
   <origin xyz="0.006213 -0.1 0.10975" rpy="0 0 0"/>
   <parent link="lazer_alt_v1_1"/>
@@ -365,19 +365,17 @@
   <limit upper="0.523599" lower="-0.261799" effort="100" velocity="100"/>
 </joint>
-<joint name="sag_kol" type="revolute">
+<joint name="sag_kol" type="fixed">
   <origin xyz="-0.002 -0.39 0.175" rpy="0 0 0"/>
   <parent link="base_link"/>
   <child link="sag_montaj_v1__1__1"/>
   <axis xyz="0.0 -1.0 0.0"/>
-  <limit upper="0.174533" lower="-0.174533" effort="100" velocity="100"/>
-</joint>
-<joint name="sol_kol" type="revolute">
+</joint>
+<joint name="sol_kol" type="fixed">
   <origin xyz="-0.001 0.389 0.175762" rpy="0 0 0"/>
   <parent link="base_link"/>
   <child link="sol_montaj_1_v81_v1__1__1"/>
   <axis xyz="0.0 1.0 0.0"/>
-  <limit upper="0.174533" lower="-0.174533" effort="100" velocity="100"/>
-</joint>
-<joint name="sag_on_kol" type="revolute">
+</joint>
+<joint name="sag_on_kol" type="fixed">
   <origin xyz="0.273451 -0.031 -0.138651" rpy="0 0 0"/>
   <parent link="sag_montaj_v1__1__1"/>
@@ -386,5 +384,5 @@
   <limit upper="0.174533" lower="-0.174533" effort="100" velocity="100"/>
 </joint>
-<joint name="sol_on_kol" type="revolute">
+<joint name="sol_on_kol" type="fixed">
   <origin xyz="0.273451 0.031 -0.13865" rpy="0 0 0"/>
   <parent link="sol_montaj_1_v81_v1__1__1"/>

File: src/ika_description/urdf/rplidar_s2.xacro (robot description, xacro)
@@ -57,10 +57,10 @@
               <samples>360</samples>
               <resolution>1</resolution>
-              <min_angle>-1.046</min_angle>
-              <max_angle>1.046</max_angle>
+              <min_angle>-3.14159</min_angle>
+              <max_angle>3.14159</max_angle>
             </horizontal>
           </scan>
           <range>
-            <min>0.2</min>
+            <min>0.6</min>
             <max>20.0</max>
             <resolution>0.02</resolution>
@@ -72,13 +72,13 @@
           </noise>
         </ray>
-        <update_rate>10.0</update_rate>
+        <update_rate>20.0</update_rate>
         <visualize>true</visualize>
         <plugin name="${name}_laser_controller" filename="libgazebo_ros_ray_sensor.so">
           <ros>
-            <remapping>~/out:=/ika/scan</remapping>
+            <remapping>~/out:=/scan</remapping>
           </ros>
           <output_type>sensor_msgs/LaserScan</output_type>
           <frame_name>${name}_laser_frame</frame_name>
-          <min_range>0.2</min_range>
+          <min_range>0.6</min_range>
           <max_range>20.0</max_range>
           <range_resolution>0.02</range_resolution>
